Commit message: Added foot contact sensor; Fix imu location; Using joint trajectory controller; fix rviz visualization due joint trajectory controller

File: bioloid_description/gazebo.xacro (robot description, xacro)
@@ -6,15 +6,55 @@
             <robotNamespace>/typea</robotNamespace>
             <robotSimType>gazebo_ros_control/DefaultRobotHWSim</robotSimType>
-             <legacyModeNS>true</legacyModeNS>
+            <legacyModeNS>true</legacyModeNS>
         </plugin>
-		<plugin name="imu_plugin" filename="libgazebo_ros_imu.so">
-		    <alwaysOn>true</alwaysOn>
-		    <bodyName>imu_link</bodyName>
-		    <topicName>/typea/imu</topicName>
-		    <serviceName>imu_service</serviceName>
-		    <gaussianNoise>0.0</gaussianNoise>
-		    <updateRate>20.0</updateRate>
-		    <visualize>true</visualize>
-		</plugin>
+        <plugin name="imu_plugin" filename="libgazebo_ros_imu.so">
+            <alwaysOn>true</alwaysOn>
+            <bodyName>imu_link</bodyName>
+            <topicName>/typea/imu</topicName>
+            <serviceName>imu_service</serviceName>
+            <gaussianNoise>0.0</gaussianNoise>
+            <updateRate>30.0</updateRate>
+            <visualize>true</visualize>
+        </plugin>
+    </gazebo>
+    <!-- Right and Left Contact Sensors -->
+    <gazebo reference="l_contact_sensor_link">
+        <sensor name="footl_contact_sensor" type="contact">
+            <always_on>true</always_on>
+            <update_rate>30</update_rate>
+            <contact>
+                <collision>l_ankle_lateral_link_fixed_joint_lump__l_contact_sensor_link_collision_2</collision>
+            </contact>
+            <plugin name="gazebo_ros_bumper_l_controller" filename="libgazebo_ros_bumper.so">
+                <bumperTopicName>/typea/footl_contact_sensor_state</bumperTopicName>
+                <frameName>l_contact_sensor_link</frameName>
+            </plugin>
+        </sensor>
+    </gazebo>
+    <gazebo reference="r_contact_sensor_link">
+        <sensor name="footr_contact_sensor" type="contact">
+            <always_on>true</always_on>
+            <update_rate>30</update_rate>
+            <contact>
+                <collision>r_ankle_lateral_link_fixed_joint_lump__r_contact_sensor_link_collision_2</collision>
+            </contact>
+            <plugin name="gazebo_ros_bumper_r_controller" filename="libgazebo_ros_bumper.so">
+                <bumperTopicName>/typea/footr_contact_sensor_state</bumperTopicName>
+                <frameName>r_contact_sensor_link</frameName>
+            </plugin>
+        </sensor>
+    </gazebo>
+    <!-- Ground Truth Pose -->
+    <gazebo>
+        <plugin name="ground_truth" filename="libgazebo_ros_p3d.so">
+            <alwaysOn>true</alwaysOn>
+            <updateRate>30.0</updateRate>
+            <bodyName>base_link</bodyName>
+            <topicName>/typea/odom</topicName>
+            <gaussianNoise>0.0</gaussianNoise>
+            <frameName>world</frameName>
+            <xyzOffsets>0 0 0</xyzOffsets>
+            <rpyOffsets>0 0 0</rpyOffsets>
+        </plugin>
     </gazebo>
     <xacro:macro name="shoulder_swing_joint_gazebo" params="prefix">

File: bioloid_description/typea.xacro (robot description, xacro)
@@ -1,20 +1,20 @@
 <?xml version="1.0"?>
 <robot xmlns:xacro="http://www.ros.org/wiki/xacro" name="typea">
-	<!-- Import mass property (inertia) -->
-	<xacro:include filename="$(find bioloid_description)/inertia/Torso.xacro"/>
-	<xacro:include filename="$(find bioloid_description)/inertia/F1.xacro"/>
-	<xacro:include filename="$(find bioloid_description)/inertia/F5.xacro"/>
-	<xacro:include filename="$(find bioloid_description)/inertia/F12.xacro"/>
-	<xacro:include filename="$(find bioloid_description)/inertia/F11.xacro"/>
-	<xacro:include filename="$(find bioloid_description)/inertia/upperarm.xacro"/>
-	<xacro:include filename="$(find bioloid_description)/inertia/upperleg.xacro"/>
-	<xacro:include filename="$(find bioloid_description)/inertia/L_Foot.xacro"/>
-	<xacro:include filename="$(find bioloid_description)/inertia/R_Foot.xacro"/>
-	<xacro:include filename="$(find bioloid_description)/inertia/L_lowerarm.xacro"/>
-	<xacro:include filename="$(find bioloid_description)/inertia/R_lowerarm.xacro"/>
-	<xacro:include filename="$(find bioloid_description)/inertia/L_Tibia.xacro"/>
-	<xacro:include filename="$(find bioloid_description)/inertia/R_Tibia.xacro"/>
-	<xacro:include filename="$(find bioloid_description)/inertia/L_hip-R_ankle.xacro"/>
-	<xacro:include filename="$(find bioloid_description)/inertia/R_hip-L_ankle.xacro"/>
+    <!-- Import mass property (inertia) -->
+    <xacro:include filename="$(find bioloid_description)/inertia/Torso.xacro"/>
+    <xacro:include filename="$(find bioloid_description)/inertia/F1.xacro"/>
+    <xacro:include filename="$(find bioloid_description)/inertia/F5.xacro"/>
+    <xacro:include filename="$(find bioloid_description)/inertia/F12.xacro"/>
+    <xacro:include filename="$(find bioloid_description)/inertia/F11.xacro"/>
+    <xacro:include filename="$(find bioloid_description)/inertia/upperarm.xacro"/>
+    <xacro:include filename="$(find bioloid_description)/inertia/upperleg.xacro"/>
+    <xacro:include filename="$(find bioloid_description)/inertia/L_Foot.xacro"/>
+    <xacro:include filename="$(find bioloid_description)/inertia/R_Foot.xacro"/>
+    <xacro:include filename="$(find bioloid_description)/inertia/L_lowerarm.xacro"/>
+    <xacro:include filename="$(find bioloid_description)/inertia/R_lowerarm.xacro"/>
+    <xacro:include filename="$(find bioloid_description)/inertia/L_Tibia.xacro"/>
+    <xacro:include filename="$(find bioloid_description)/inertia/R_Tibia.xacro"/>
+    <xacro:include filename="$(find bioloid_description)/inertia/L_hip-R_ankle.xacro"/>
+    <xacro:include filename="$(find bioloid_description)/inertia/R_hip-L_ankle.xacro"/>
     <!-- Import gazebo_ros_control plugin -->
     <xacro:include filename="$(find bioloid_description)/gazebo.xacro" ns="gazebo"/>
@@ -37,5 +37,5 @@
     <joint name="imu_to_base_joint" type="fixed">
         <axis xyz="1 0 0"/>
-        <origin xyz="0 0 0.05" rpy="0 0 0"/>
+        <origin xyz="0.0 0 0" rpy="0 0 0"/>
         <parent link="base_link"/>
         <child link="imu_link"/>
@@ -51,16 +51,82 @@
             </material>
         </visual>
-          <collision>
-	    <origin rpy="0 0 0" xyz="0 0 0"/>
-	        <geometry>
-	        <box size=".01 .01 .01"/>
-	        </geometry>
-	    </collision>
-	  <inertial>
-	    <mass value="0.001"/>
-	    <origin rpy="0 0 0" xyz="0 0 0"/>
-	    <inertia ixx="0.0001" ixy="0" ixz="0" iyy="0.000001" iyz="0" izz="0.0001"/>
-	  </inertial>
-    </link>
+        <collision>
+            <origin rpy="0 0 0" xyz="0 0 0"/>
+            <geometry>
+                <box size=".01 .01 .01"/>
+            </geometry>
+        </collision>
+        <inertial>
+            <mass value="0.001"/>
+            <origin rpy="0 0 0" xyz="0 0 0"/>
+            <inertia ixx="0.0001" ixy="0" ixz="0" iyy="0.000001" iyz="0" izz="0.0001"/>
+        </inertial>
+    </link>
+    <gazebo reference="imu_link">
+        <material>Gazebo/Red</material>
+    </gazebo>
+    <!-- Foot Contact Sensor -->
+    <joint name="l_foot_sensor_joint" type="fixed">
+        <axis xyz="0 0 0"/>
+        <origin xyz="-0.032 0 0" rpy="0 ${pi/2} 0"/>
+        <parent link="l_foot_link"/>
+        <child link="l_contact_sensor_link"/>
+    </joint>
+    <link name="l_contact_sensor_link">
+        <visual>
+            <origin rpy="0 0 0" xyz="0 0 0"/>
+            <geometry>
+                <box size="0.08 0.06 0.001"/>
+            </geometry>
+            <material name="red">
+                <color rgba="1.0 0.0 0.0 1.0"/>
+            </material>
+        </visual>
+        <collision>
+            <origin rpy="0 0 0" xyz="0 0 0"/>
+            <geometry>
+                <box size=".01 .01 .001"/>
+            </geometry>
+        </collision>
+        <!--inertial>
+            <mass value="0.001"/>
+            <origin rpy="0 0 0" xyz="0 0 0"/>
+            <inertia ixx="0.0001" ixy="0" ixz="0" iyy="0.000001" iyz="0" izz="0.0001"/>
+        </inertial-->
+    </link>
+    <gazebo reference="l_contact_sensor_link">
+        <material>Gazebo/Red</material>
+    </gazebo>
+    <joint name="r_foot_sensor_joint" type="fixed">
+        <axis xyz="0 0 0"/>
+        <origin xyz="0.032 0 0" rpy="0 ${pi/2} 0"/>
+        <parent link="r_foot_link"/>
+        <child link="r_contact_sensor_link"/>
+    </joint>
+    <link name="r_contact_sensor_link">
+        <visual>
+            <origin rpy="0 0 0" xyz="0 0 0"/>
+            <geometry>
+                <box size="0.08 0.06 0.001"/>
+            </geometry>
+            <material name="red">
+                <color rgba="1.0 0.0 0.0 1.0"/>
+            </material>
+        </visual>
+        <collision>
+            <origin rpy="0 0 0" xyz="0 0 0"/>
+            <geometry>
+                <box size=".01 .01 .001"/>
+            </geometry>
+        </collision>
+        <!--inertial>
+            <mass value="0.001"/>
+            <origin rpy="0 0 0" xyz="0 0 0"/>
+            <inertia ixx="0.0001" ixy="0" ixz="0" iyy="0.000001" iyz="0" izz="0.0001"/>
+        </inertial-->
+    </link>
+    <gazebo reference="r_contact_sensor_link">
+        <material>Gazebo/Red</material>
+    </gazebo>
     <xacro:macro name="shoulder_swing_joint" params="prefix reflect">
         <joint name="${prefix}_shoulder_swing_joint" type="revolute">
@@ -164,207 +230,208 @@
             <minDepth>0.001</minDepth>
             <maxContacts>1</maxContacts>
+            <material>Gazebo/Grey</material>
         </gazebo>
     </xacro:macro>
     <!-- Links MACRO -->
     <xacro:macro name="hip_lateral_link" params="prefix reflect x_offset y_offset z_offset *inertial">
-    <link name="${prefix}_hip_lateral_link">
-        <!-- Motor 9[r] 10[l] -->
-        <visual>
-            <default_geometry cad_file="AX-12"/>
-            <origin xyz="0 0 ${z_offset}" rpy="0 0 ${(reflect-1)*pi*-1/2}"/>
-        </visual>
-        <visual>
-            <default_geometry cad_file="FP04-F6"/>
-            <origin xyz="${-1*reflect*0.019} ${-1*reflect*0.0145} ${z_offset+0.016}" rpy="0 ${-pi/2} ${-1*reflect*pi/2}"/>
-        </visual>
-        <visual>
-            <default_geometry cad_file="FP04-F6"/>
-            <origin xyz="${reflect*0.019} ${-1*reflect*0.0145} ${z_offset+0.016}" rpy="0 ${-pi/2} ${reflect*pi/2}"/>
-        </visual>
-        <!-- Motor 11[r] 12[l] -->
-        <visual>
-            <default_geometry cad_file="AX-12"/>
-            <origin xyz="0 0 ${z_offset-0.032}" rpy="${(reflect-1)*pi*-1/2} ${-1*reflect*pi/2} 0"/>
-        </visual>
-        <visual>
-            <default_geometry cad_file="BPF-BU"/>
-            <origin xyz="0 0 ${z_offset-0.05}" rpy="${-1*reflect*pi/2} ${(reflect-1)*pi*-1/2} 0"/>
-        </visual>
-        <visual>
-            <default_geometry cad_file="FP04-F7"/>
-            <origin xyz="0 ${-1*reflect*0.0145} ${z_offset-0.051}" rpy="${reflect*pi/2} ${(reflect-1)*pi*-1/2} ${pi/2}"/>
-        </visual>
-        <collision name="r_hip_lateral_collision">
-            <origin xyz="0 ${-1*reflect*0.0135} ${z_offset-0.0153}"/>
-            <geometry>
-                <box size="0.04 0.051 0.0721"/>
-            </geometry>
-        </collision>
-        <xacro:insert_block name="inertial" />
-        <!--
+        <link name="${prefix}_hip_lateral_link">
+            <!-- Motor 9[r] 10[l] -->
+            <visual>
+                <default_geometry cad_file="AX-12"/>
+                <origin xyz="0 0 ${z_offset}" rpy="0 0 ${(reflect-1)*pi*-1/2}"/>
+            </visual>
+            <visual>
+                <default_geometry cad_file="FP04-F6"/>
+                <origin xyz="${-1*reflect*0.019} ${-1*reflect*0.0145} ${z_offset+0.016}" rpy="0 ${-pi/2} ${-1*reflect*pi/2}"/>
+            </visual>
+            <visual>
+                <default_geometry cad_file="FP04-F6"/>
+                <origin xyz="${reflect*0.019} ${-1*reflect*0.0145} ${z_offset+0.016}" rpy="0 ${-pi/2} ${reflect*pi/2}"/>
+            </visual>
+            <!-- Motor 11[r] 12[l] -->
+            <visual>
+                <default_geometry cad_file="AX-12"/>
+                <origin xyz="0 0 ${z_offset-0.032}" rpy="${(reflect-1)*pi*-1/2} ${-1*reflect*pi/2} 0"/>
+            </visual>
+            <visual>
+                <default_geometry cad_file="BPF-BU"/>
+                <origin xyz="0 0 ${z_offset-0.05}" rpy="${-1*reflect*pi/2} ${(reflect-1)*pi*-1/2} 0"/>
+            </visual>
+            <visual>
+                <default_geometry cad_file="FP04-F7"/>
+                <origin xyz="0 ${-1*reflect*0.0145} ${z_offset-0.051}" rpy="${reflect*pi/2} ${(reflect-1)*pi*-1/2} ${pi/2}"/>
+            </visual>
+            <collision name="r_hip_lateral_collision">
+                <origin xyz="0 ${-1*reflect*0.0135} ${z_offset-0.0153}"/>
+                <geometry>
+                    <box size="0.04 0.051 0.0721"/>
+                </geometry>
+            </collision>
+            <xacro:insert_block name="inertial" />
+            <!--
         <inertial>
             <origin xyz="0.000079 0.018242 0.013873" />
             <mass value="0.11904336"/>
-            <inertia ixx="0.097950272"  ixy="0.0012119368"  ixz="-0.00021223016" iyx="0.00122119368" iyy="0.032848287" iyz="-0.0019474021" izx="-0.00021223016" izy="-0.0019474021" izz="0.11493509" />
-        </inertial>
-        -->
-    </link>
+            <inertia ixx="0.097950272" ixy="0.0012119368" ixz="-0.00021223016" iyx="0.00122119368" iyy="0.032848287" iyz="-0.0019474021" izx="-0.00021223016" izy="-0.0019474021" izz="0.11493509" />
+        </inertial>
+        -->
+        </link>
     </xacro:macro>
     <xacro:macro name="hip_twist_link" params="prefix reflect x_offset y_offset z_offset">
-    <link name="${prefix}_hip_twist_link">
-        <visual>
-            <default_geometry cad_file="FP04-F5"/>
-            <origin xyz="0 ${reflect*y_offset} 0.05" rpy="${pi} 0 ${(reflect+1)*pi*1/2}"/>
-        </visual>
-        <collision name="r_hip_twist_collision">
-            <origin xyz="0.0008 ${reflect*y_offset} 0.041"/>
-            <geometry>
-                <box size="0.029 0.083 0.0405"/>
-            </geometry>
-        </collision>
-        <xacro:hip_twist_inertial/>
-        <!--
+        <link name="${prefix}_hip_twist_link">
+            <visual>
+                <default_geometry cad_file="FP04-F5"/>
+                <origin xyz="0 ${reflect*y_offset} 0.05" rpy="${pi} 0 ${(reflect+1)*pi*1/2}"/>
+            </visual>
+            <collision name="r_hip_twist_collision">
+                <origin xyz="0.0008 ${reflect*y_offset} 0.041"/>
+                <geometry>
+                    <box size="0.029 0.083 0.0405"/>
+                </geometry>
+            </collision>
+            <xacro:hip_twist_inertial/>
+            <!--
         <inertial>
             <origin xyz="0.000000 0.000480 0.018437" />
             <mass value="0.167"/>
-            <inertia ixx="0.12259691"  ixy="0.00071127469"  ixz="0.00081143913" iyx="0.00071127469" iyy="0.11066637" iyz="-0.0071635476" izx="0.00081143913" izy="-0.0071635476" izz="0.041877668" />
-        </inertial>
-        -->
-    </link>
+            <inertia ixx="0.12259691" ixy="0.00071127469" ixz="0.00081143913" iyx="0.00071127469" iyy="0.11066637" iyz="-0.0071635476" izx="0.00081143913" izy="-0.0071635476" izz="0.041877668" />
+        </inertial>
+        -->
+        </link>
     </xacro:macro>
     <xacro:macro name="upper_leg_link" params="prefix reflect x_offset y_offset z_offset">
-    <link name="${prefix}_upper_leg_link">
-        <visual>
-            <default_geometry cad_file="FP04-F4"/>
-            <origin xyz="0 0 0" rpy="${-1*reflect*pi/2} ${-1*reflect*pi/2} ${-pi/2}"/>
-        </visual>
-        <visual>
-            <default_geometry cad_file="FP04-F1"/>
-            <origin xyz="${reflect*0.075} 0.0145 0" rpy="${pi/2} ${reflect*pi/2} ${-1*reflect*pi/2}"/>
-        </visual>
-        <collision name="r_upper_leg_proximal_collision">
-            <origin xyz="${reflect*0.0214} 0 0"/>
-            <geometry>
-                <box size="0.065 0.03 0.049"/>
-            </geometry>
-        </collision>
-        <collision name="r_upper_leg_distal_collision">
-            <origin xyz="${reflect*0.0675} 0.0065 0"/>
-            <geometry>
-                <box size="0.04 0.0371 0.049"/>
-            </geometry>
-        </collision>
-        <xacro:upperleg_inertial/>
-        <!--
+        <link name="${prefix}_upper_leg_link">
+            <visual>
+                <default_geometry cad_file="FP04-F4"/>
+                <origin xyz="0 0 0" rpy="${-1*reflect*pi/2} ${-1*reflect*pi/2} ${-pi/2}"/>
+            </visual>
+            <visual>
+                <default_geometry cad_file="FP04-F1"/>
+                <origin xyz="${reflect*0.075} 0.0145 0" rpy="${pi/2} ${reflect*pi/2} ${-1*reflect*pi/2}"/>
+            </visual>
+            <collision name="r_upper_leg_proximal_collision">
+                <origin xyz="${reflect*0.0214} 0 0"/>
+                <geometry>
+                    <box size="0.065 0.03 0.049"/>
+                </geometry>
+            </collision>
+            <collision name="r_upper_leg_distal_collision">
+                <origin xyz="${reflect*0.0675} 0.0065 0"/>
+                <geometry>
+                    <box size="0.04 0.0371 0.049"/>
+                </geometry>
+            </collision>
+            <xacro:upperleg_inertial/>
+            <!--
         <inertial>
             <origin xyz="-0.062965 -0.000323 0.000692" />
             <mass value="0.11904336"/>
-            <inertia ixx="0.097950272"  ixy="0.0012119368"  ixz="-0.00021223016" iyx="0.00122119368" iyy="0.032848287" iyz="-0.0019474021" izx="-0.00021223016" izy="-0.0019474021" izz="0.11493509" />
-        </inertial>
-        -->
-    </link>
+            <inertia ixx="0.097950272" ixy="0.0012119368" ixz="-0.00021223016" iyx="0.00122119368" iyy="0.032848287" iyz="-0.0019474021" izx="-0.00021223016" izy="-0.0019474021" izz="0.11493509" />
+        </inertial>
+        -->
+        </link>
     </xacro:macro>
     <xacro:macro name="lower_leg_link" params="prefix reflect x_offset y_offset z_offset *inertial">
-    <link name="${prefix}_lower_leg_link">
-        <!-- Motor 13[r] 14[l] -->
-        <visual>
-            <default_geometry cad_file="AX-12"/>
-            <origin xyz="0 0 0" rpy="0 0 0"/>
-        </visual>
-        <visual>
-            <default_geometry cad_file="FP04-F3"/>
-            <origin xyz="${reflect*0.019} -0.0145 0" rpy="0 0 ${reflect*pi/2}"/>
-        </visual>
-        <visual>
-            <default_geometry cad_file="FP04-F4"/>
-            <origin xyz="${reflect*0.071} -0.0145 0" rpy="${reflect*pi/2} ${reflect*pi/2} ${-pi/2}"/>
-        </visual>
-        <collision name="r_lower_leg_proximal_collision">
-            <origin xyz="0 -0.0135 0"/>
-            <geometry>
-                <box size="0.033 0.051 0.044"/>
-            </geometry>
-        </collision>
-        <collision name="r_lower_leg_distal_collision">
-            <origin xyz="${reflect*0.0492} -0.0145 0"/>
-            <geometry>
-                <box size="0.067 0.03 0.049"/>
-            </geometry>
-        </collision>
-        <xacro:insert_block name="inertial" />
-        <!--
+        <link name="${prefix}_lower_leg_link">
+            <!-- Motor 13[r] 14[l] -->
+            <visual>
+                <default_geometry cad_file="AX-12"/>
+                <origin xyz="0 0 0" rpy="0 0 0"/>
+            </visual>
+            <visual>
+                <default_geometry cad_file="FP04-F3"/>
+                <origin xyz="${reflect*0.019} -0.0145 0" rpy="0 0 ${reflect*pi/2}"/>
+            </visual>
+            <visual>
+                <default_geometry cad_file="FP04-F4"/>
+                <origin xyz="${reflect*0.071} -0.0145 0" rpy="${reflect*pi/2} ${reflect*pi/2} ${-pi/2}"/>
+            </visual>
+            <collision name="r_lower_leg_proximal_collision">
+                <origin xyz="0 -0.0135 0"/>
+                <geometry>
+                    <box size="0.033 0.051 0.044"/>
+                </geometry>
+            </collision>
+            <collision name="r_lower_leg_distal_collision">
+                <origin xyz="${reflect*0.0492} -0.0145 0"/>
+                <geometry>
+                    <box size="0.067 0.03 0.049"/>
+                </geometry>
+            </collision>
+            <xacro:insert_block name="inertial" />
+            <!--
         <inertial>
             <origin xyz="-0.053955 0.006548 -0.000592" />
             <mass value="0.070309794"/>
-            <inertia ixx="0.093369608"  ixy="-0.00093567395"  ixz="-0.00023992085" iyx="-0.00093567395" iyy="0.046295534" iyz="-0.012858493" izx="-0.00023992085" izy="-0.012858493" izz="0.11351516" />
-        </inertial>
-        -->
-    </link>
+            <inertia ixx="0.093369608" ixy="-0.00093567395" ixz="-0.00023992085" iyx="-0.00093567395" iyy="0.046295534" iyz="-0.012858493" izx="-0.00023992085" izy="-0.012858493" izz="0.11351516" />
+        </inertial>
+        -->
+        </link>
     </xacro:macro>
     <xacro:macro name="ankle_swing_link" params="prefix reflect x_offset y_offset z_offset *inertial">
-    <link name="${prefix}_ankle_swing_link">
-        <!-- Motor 15[r] 16[l] -->
-        <visual>
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